Commit message: menambahkan sensor IMU pada file urdf robot

File: my_robot/urdf/my_robot.urdf.xacro (robot description, xacro)
@@ -69,4 +69,19 @@
     <origin xyz="0.12 0 -0.03" rpy="0 0 0"/>
   </joint>
+  <!-- IMU LINK & SENSOR -->
+  <link name="imu_link"/>
+  <joint name="imu_joint" type="fixed">
+    <parent link="base_link"/>
+    <child link="imu_link"/>
+    <origin xyz="0 0 0" rpy="0 0 0"/>
+  </joint>
+  <gazebo reference="imu_link">
+    <sensor name="imu_sensor" type="imu">
+      <always_on>1</always_on>
+      <update_rate>100</update_rate>
+      <visualize>true</visualize>
+      <topic>imu</topic>
+    </sensor>
+  </gazebo>
   <!-- GAZEBO PLUGINS -->
   <gazebo>
@@ -88,4 +103,5 @@
       <joint_name>right_wheel_joint</joint_name>
     </plugin>
+    <plugin filename="gz-sim-imu-system" name="gz::sim::systems::Imu"/>
   </gazebo>
   <gazebo reference="caster_wheel">
